File: hardware/ghost-feather-v1/ghost-feather-v1.kicad_pcb (KiCad board)
At the start: 4 copper layers, 106.6 x 106.7 mm, 72 parts, among them J1 Conn_ARM_SWD_TagConnect_TC2030, J2 USB_C_Receptacle_USB2.0, J3 Conn_01x03, J4 Conn_01x03, J5 Conn_01x03, J6 Conn_01x03, J7 Conn_01x08, Q1 BSS138, Q2 BSS138, Q3 BSS138, Q4 BSS138, SW2 BOOT0, U1 STM32F722RETx, U2 BMI270, U3 USBLC6-2SC6_MOD, U4 MPM3610, U5 MPM3610, X1 16MHz, X2 32kHz768

Commit message: feat: PCB routing #2
Parts:
- moved D3 6.38 mm to (171.6, 109.0), turned to -90 degrees
- moved R27 6.38 mm to (165.9, 106.0), turned to -90 degrees
- moved C20 0.12 mm to (175.4, 104.5)
- moved R24 0.12 mm to (174.0, 104.8)
Routing:
- net Net-(U4-FB): track 0.00 -> 10.4 mm
- net Net-(U5-FB): track 0.00 -> 10.3 mm
- net +BATT: track 0.00 -> 3.27 mm
- net +5V: track 0.00 -> 3.15 mm
- net GND: track 39.0 -> 41.0 mm
- net Net-(U4-EN): track 0.00 -> 1.56 mm
- net Net-(U5-EN): track 0.00 -> 1.38 mm
- net Net-(U4-AAM): track 0.00 -> 1.32 mm
- net Net-(U5-AAM): track 0.00 -> 1.30 mm
- net Net-(D3-A): track 0.00 -> 1.18 mm
- net Net-(D2-A): track 0.00 -> 1.16 mm

Commit message: feat: PCB routing #3
Parts:
- moved J1 11.2 mm to (124.7, 81.0)
- turned U3 to 0 degrees
Connections:
- net /USBC_DM renamed /USBC_D-
- net /USBC_DP renamed /USBC_D+
- net /USB_DM renamed /USB_D-
- net /USB_DP renamed /USB_D+
Routing:
- net /USB_D-: track 0.00 -> 19.5 mm
- net /USB_D+: track 0.00 -> 19.5 mm
- net /USBC_D-: track 0.00 -> 18.7 mm
- net /USBC_D+: track 0.00 -> 17.6 mm
- net Net-(J2-CC1): track 0.00 -> 7.73 mm
- net Net-(J2-CC2): track 0.00 -> 7.17 mm

Commit message: feat: PCB routing #4
Parts:
- moved J1 32.8 mm to (142.9, 108.3)
- moved C10 13.9 mm to (131.1, 98.3), turned to 0 degrees
- moved SW2 13.8 mm to (125.8, 95.1)
- moved R2 13.3 mm to (130.6, 95.6), turned to 90 degrees
- moved R1 13.2 mm to (131.1, 97.2), turned to 180 degrees
- moved C9 0.10 mm to (149.9, 91.2)
Routing:
- net /SWD_NRST: track 2.44 -> 33.7 mm, vias 0 -> 2
- net /SWD_DIO: track 0.00 -> 19.9 mm, vias 0 -> 2
- net /SWD_TRC: track 0.00 -> 15.2 mm
- net /BOOT0: track 7.47 -> 22.4 mm, vias 0 -> 2
- net /SWD_CLK: track 0.00 -> 11.8 mm
- added copper zone on F.Cu, net /ESC0
- added copper zone on F.Cu, net /ESC1
- added copper zone on F.Cu, net /ESC2
- added copper zone on F.Cu, net /ESC3

Commit message: feat: PCB routing #5
Routing:
- net +3V3: track 14.6 -> 20.8 mm, vias 0 -> 19
- net GND: track 41.0 -> 45.8 mm, vias 52 -> 64
- net Net-(J4-Pin_2): track 0.00 -> 3.89 mm
- net Net-(J5-Pin_2): track 0.00 -> 3.87 mm
- net Net-(J3-Pin_2): track 0.00 -> 3.86 mm
- net Net-(J6-Pin_2): track 0.00 -> 3.77 mm
- net +5V: vias 0 -> 8
- added copper zone on B.Cu, net +3V3
- added copper zone on F.Cu, net +3V3
- added copper zone on F.Cu, net +5V
- added copper zone on F.Cu, net GND
- added copper zone on In1.Cu, net GND
- added copper zone on In2.Cu, net GND
- removed copper zone on B.Cu, net GND

Commit message: feat: PCB routing #6
Parts:
- moved D1 1.11 mm to (150.6, 84.7)
- moved R15 1.11 mm to (150.6, 85.9)
- moved C17 0.07 mm to (117.1, 123.2)
- moved Q1 0.07 mm to (113.7, 121.2)
- moved R12 0.07 mm to (111.7, 117.8)
- moved R13 0.07 mm to (112.6, 118.7)
- moved R14 0.07 mm to (116.2, 122.3)
Routing:
- net +5V: track 3.15 -> 346.4 mm, vias 8 -> 18
- net +3V3: track 20.8 -> 31.3 mm, vias 19 -> 35
- net /BMI270_CSB: track 3.36 -> 11.9 mm, vias 0 -> 2
- net Net-(J6-Pin_2): track 3.77 -> 7.18 mm
- net Net-(J4-Pin_2): track 3.89 -> 7.23 mm
- net Net-(J3-Pin_2): track 3.86 -> 7.13 mm
- net Net-(J5-Pin_2): track 3.87 -> 6.89 mm
- net /LED_USER: track 2.89 -> 4.02 mm
- net GND: vias 64 -> 68

Commit message: feat: PCB routing #7
Routing:
- net GND: vias 68 -> 82
Changed lines of the file:
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@@
   (segment (start 168.033411 61.133411) (end 167.3 60.4) (width 0.3) (layer "F.Cu") (net 2))
   (segment (start 159.28 97.33) (end 159.275 97.325) (width 0.3) (layer "F.Cu") (net 2))
+  (via (at 145.7 95.65) (size 0.8) (drill 0.4) (layers "F.Cu" "B.Cu") (free) (net 2))
   (via (at 149.0725 84.665) (size 0.8) (drill 0.4) (layers "F.Cu" "B.Cu") (free) (net 2))
+  (via (at 143.7 95.65) (size 0.8) (drill 0.4) (layers "F.Cu" "B.Cu") (free) (net 2))
+  (via (at 140.25 89.55) (size 0.8) (drill 0.4) (layers "F.Cu" "B.Cu") (free) (net 2))
   (via (at 159.275 99.675) (size 0.8) (drill 0.4) (layers "F.Cu" "B.Cu") (free) (net 2))
   (via (at 176.7 63.175) (size 0.8) (drill 0.4) (layers "F.Cu" "B.Cu") (free) (net 2))
@@
   (via (at 175.9 79.35) (size 0.8) (drill 0.4) (layers "F.Cu" "B.Cu") (free) (net 2))
   (via (at 132.6 98.35) (size 0.8) (drill 0.4) (layers "F.Cu" "B.Cu") (free) (net 2))
+  (via (at 141.25 88.05) (size 0.8) (drill 0.4) (layers "F.Cu" "B.Cu") (free) (net 2))
+  (via (at 142.5 89.5) (size 0.8) (drill 0.4) (layers "F.Cu" "B.Cu") (free) (net 2))
+  (via (at 143.75 88.05) (size 0.8) (drill 0.4) (layers "F.Cu" "B.Cu") (free) (net 2))
+  (via (at 145.75 88.05) (size 0.8) (drill 0.4) (layers "F.Cu" "B.Cu") (free) (net 2))
   (via (at 114.325 58.075) (size 0.8) (drill 0.4) (layers "F.Cu" "B.Cu") (free) (net 2))
   (via (at 165.95 107.5) (size 0.8) (drill 0.4) (layers "F.Cu" "B.Cu") (free) (net 2))
@@
   (via (at 138.73 82.56) (size 0.8) (drill 0.4) (layers "F.Cu" "B.Cu") (free) (net 2))
   (via (at 170.425 125.475) (size 0.8) (drill 0.4) (layers "F.Cu" "B.Cu") (free) (net 2))
+  (via (at 140.2 94.2) (size 0.8) (drill 0.4) (layers "F.Cu" "B.Cu") (free) (net 2))
   (via (at 172.55 85.2) (size 0.8) (drill 0.4) (layers "F.Cu" "B.Cu") (free) (net 2))
+  (via (at 142.45 94.2) (size 0.8) (drill 0.4) (layers "F.Cu" "B.Cu") (free) (net 2))
   (via (at 173.7 101.75) (size 0.8) (drill 0.4) (layers "F.Cu" "B.Cu") (free) (net 2))
   (via (at 109.65 119.975) (size 0.8) (drill 0.4) (layers "F.Cu" "B.Cu") (free) (net 2))
@@
   (via (at 167.3 60.4) (size 0.8) (drill 0.4) (layers "F.Cu" "B.Cu") (free) (net 2))
   (via (at 114.9 91.3) (size 0.8) (drill 0.4) (layers "F.Cu" "B.Cu") (free) (net 2))
+  (via (at 141.2 95.65) (size 0.8) (drill 0.4) (layers "F.Cu" "B.Cu") (free) (net 2))
   (via (at 172.67 108.45) (size 0.8) (drill 0.4) (layers "F.Cu" "B.Cu") (free) (net 2))
   (via (at 171.775 126.85) (size 0.8) (drill 0.4) (layers "F.Cu" "B.Cu") (free) (net 2))
   (via (at 159.275 97.325) (size 0.8) (drill 0.4) (layers "F.Cu" "B.Cu") (free) (net 2))
+  (via (at 139.2 95.65) (size 0.8) (drill 0.4) (layers "F.Cu" "B.Cu") (free) (net 2))
+  (via (at 144.75 89.5) (size 0.8) (drill 0.4) (layers "F.Cu" "B.Cu") (free) (net 2))
   (via (at 168.1 102.875) (size 0.8) (drill 0.4) (layers "F.Cu" "B.Cu") (free) (net 2))
   (via (at 108.275 121.325) (size 0.8) (drill 0.4) (layers "F.Cu" "B.Cu") (free) (net 2))
@@
   (via (at 113.625 57.4) (size 0.8) (drill 0.4) (layers "F.Cu" "B.Cu") (free) (net 2))
   (via (at 165.825 85.15) (size 0.8) (drill 0.4) (layers "F.Cu" "B.Cu") (free) (net 2))
+  (via (at 139.25 88.05) (size 0.8) (drill 0.4) (layers "F.Cu" "B.Cu") (free) (net 2))
   (via (at 173.6 83.4) (size 0.8) (drill 0.4) (layers "F.Cu" "B.Cu") (free) (net 2))
   (via (at 108.95 120.625) (size 0.8) (drill 0.4) (layers "F.Cu" "B.Cu") (free) (net 2))
@@
   (via (at 114.3 59.475) (size 0.8) (drill 0.4) (layers "F.Cu" "B.Cu") (free) (net 2))
   (via (at 171.1 124.775) (size 0.8) (drill 0.4) (layers "F.Cu" "B.Cu") (free) (net 2))
+  (via (at 144.7 94.15) (size 0.8) (drill 0.4) (layers "F.Cu" "B.Cu") (free) (net 2))
   (via (at 165.95 108.45) (size 0.8) (drill 0.4) (layers "F.Cu" "B.Cu") (free) (net 2))
   (via (at 146.28 83.45) (size 0.8) (drill 0.4) (layers "F.Cu" "B.Cu") (free) (net 2))

Commit message: feat: PCB routing #8. PCB cleanup #1
Parts:
- removed G***: LOGO, ghost-feather-v1:f450_04192025
- added FID1: Fiducial, Fiducial:Fiducial_1.5mm_Mask4.5mm, F.Cu at (101.2, 58.7)
- added FID2: Fiducial, Fiducial:Fiducial_1.5mm_Mask4.5mm, F.Cu at (109.8, 50.2)
- added FID3: Fiducial, Fiducial:Fiducial_1.5mm_Mask4.5mm, F.Cu at (175.4, 50.7)
- added FID4: Fiducial, Fiducial:Fiducial_1.5mm_Mask4.5mm, F.Cu at (183.9, 59.3)
- added FID5: Fiducial, Fiducial:Fiducial_1.5mm_Mask4.5mm, F.Cu at (184.3, 125.6)
- added FID6: Fiducial, Fiducial:Fiducial_1.5mm_Mask4.5mm, F.Cu at (175.7, 134.0)
- added FID7: Fiducial, Fiducial:Fiducial_1.5mm_Mask4.5mm, F.Cu at (109.6, 133.8)
- added FID8: Fiducial, Fiducial:Fiducial_1.5mm_Mask4.5mm, F.Cu at (101.1, 125.2)
- added H1: MountingHole, MountingHole:MountingHole_2.7mm_M2.5, F.Cu at (95.5, 60.5)
- added H10: MountingHole, MountingHole:MountingHole_2.7mm_M2.5, F.Cu at (173.7, 139.3)
- added H11: MountingHole, MountingHole:MountingHole_2.7mm_M2.5, F.Cu at (162.3, 122.9)
- added H12: MountingHole, MountingHole:MountingHole_2.7mm_M2.5, F.Cu at (173.3, 111.4)
- added H13: MountingHole, MountingHole:MountingHole_2.7mm_M2.5, F.Cu at (112.0, 139.1)
- added H14: MountingHole, MountingHole:MountingHole_2.7mm_M2.5, F.Cu at (95.7, 123.2)
- added H15: MountingHole, MountingHole:MountingHole_2.7mm_M2.5, F.Cu at (112.0, 112.0)
- added H16: MountingHole, MountingHole:MountingHole_2.7mm_M2.5, F.Cu at (123.5, 123.0)
- added H2: MountingHole, MountingHole:MountingHole_2.7mm_M2.5, F.Cu at (111.3, 44.3)
- added H3: MountingHole, MountingHole:MountingHole_2.7mm_M2.5, F.Cu at (122.5, 60.6)
- added H4: MountingHole, MountingHole:MountingHole_2.7mm_M2.5, F.Cu at (111.5, 72.1)
- added H5: MountingHole, MountingHole:MountingHole_2.7mm_M2.5, F.Cu at (173.2, 45.2)
- added H6: MountingHole, MountingHole:MountingHole_2.7mm_M2.5, F.Cu at (189.4, 61.0)
- added H7: MountingHole, MountingHole:MountingHole_2.7mm_M2.5, F.Cu at (173.1, 72.3)
- added H8: MountingHole, MountingHole:MountingHole_2.7mm_M2.5, F.Cu at (161.6, 61.3)
- added H9: MountingHole, MountingHole:MountingHole_2.7mm_M2.5, F.Cu at (189.5, 123.1)
- added J8: Conn_01x02, Connector_AMASS:AMASS_XT60PW-M_1x02_P7.20mm_Horizontal, F.Cu at (182.2, 88.0)
- moved C21 1.67 mm to (168.1, 106.8)
- moved R24 1.67 mm to (173.9, 103.1)
- moved R26 1.67 mm to (167.0, 104.4)
- moved R28 1.67 mm to (170.4, 107.3)
- moved C20 1.67 mm to (175.4, 102.8)
- moved D3 1.67 mm to (171.6, 107.3)
- moved R25 1.67 mm to (173.1, 101.1)
- moved R27 1.67 mm to (165.9, 104.3)
- moved U5 1.67 mm to (170.0, 103.8)
Routing:
- net +BATT: track 3.27 -> 22.7 mm
- net GND: track 45.8 -> 57.6 mm, vias 82 -> 86
- net +5V: track 346.4 -> 352.3 mm, vias 18 -> 0

Commit message: feat: PCB cleanup #2. Via stiching #1
Routing:
- net GND: vias 86 -> 329
Other:
- board text added: "BOOT"
- board text added: "ESC0"
- board text added: "ESC1"
- board text added: "ESC2"
- board text added: "ESC3"
- board text added: "GND CH5 CH4 CH3 CH2 CH1 CH0 +5V"
- board text added: "USBC"
