File: hardware/ghost-feather-v2/kicad/ghost-feather-v2/ghost-feather-v2.kicad_sch (KiCad schematic)
At the start: 42 parts, among them J1 STM32F722RETx, J2 nRF52810, SW1 BOOT0, U1 STM32F722RETx, U2 BMI088, U2 nRF52810-QCxx, U3 IIS2MDCTR, U4 BMP390

Commit message: feat: hardware: Add crystals for nRF52810. Add voltage level shifters for ESCs
Parts:
- added C16, C17, C29, C30: 12p, symbol Device:C_Small
- added C31, C32, C33, C34: 100n, symbol Device:C_Small
- added J3, J4, J5, J6: Conn_01x03, symbol Connector_Generic:Conn_01x03
- added Q1, Q2, Q3, Q4: BSS138, Package_TO_SOT_SMD:SOT-23, symbol Transistor_FET:BSS138
- added R10, R12, R14, R3: 220, symbol Device:R_Small
- added R11, R13, R15, R16, R17, R18, R2, R6: 4k7, symbol Device:R_Small
- added X3: 32MHz, symbol Device:Crystal
- added X4: 32.768kHz, symbol Device:Crystal_Small
Connections:
- net +3V3: now also Q1.1 (G), Q2.1 (G), Q3.1 (G), Q4.1 (G), R10.2, R11.1, R12.2, R13.1, R14.2, R2.1, R3.2, R6.1
- net ESC0: now also Q1.3 (D), R2.2, R3.1
- net ESC1: now also Q2.3 (D), R10.1, R6.2
- net ESC2: now also Q3.3 (D), R11.2, R12.1
- net ESC3: now also Q4.3 (D), R13.2, R14.1
- net GND: now also C16.1, C17.1, C29.2, C30.2, C31.2, C32.2, C33.2, C34.2, J3.1 (Pin_1), J4.1 (Pin_1), J5.1 (Pin_1), J6.1 (Pin_1)
- net at U2.2 (P0.00/XL1): now also C30.1, X4.2
- net at U2.23 (XC1): now also C16.2, X3.2
- net at U2.24 (XC2): now also C17.2, X3.1
- net at U2.3 (P0.01/XL2): now also C29.1, X4.1
- new net: J4.2 (Pin_2), Q2.2 (S), R16.2
- new net: J6.2 (Pin_2), Q4.2 (S), R18.2
- new net: J3.2 (Pin_2), Q1.2 (S), R17.2
- new net: J5.2 (Pin_2), Q3.2 (S), R15.2
- new net +5V: C31.1, C32.1, C33.1, C34.1, J3.3 (Pin_3), J4.3 (Pin_3), J5.3 (Pin_3), J6.3 (Pin_3), R15.1, R16.1, R17.1, R18.1
Other:
- note added: "MICROCONTROLLERS"
- note added: "TAG CONNECTORS"
- note added: "VOLTAGE LEVEL SHIFTERS"
- note removed: "MCU"
- moved on the sheet: C10, C11, C12, C13, C14, C15, C18, C19, C23, C24, C25, C26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
